Commit message: minor updates

File: urdf/mobile.urdf (robot description, URDF)
Before this commit: robot mobile_bot, 12 links, 11 joints
Links:
- removed link bin_green
- removed link bin_red
Joints:
- removed joint bin_joint_one
- removed joint bin_joint_two

File: urdf/mobile_bot.urdf.xacro (robot description, xacro)
@@ -91,32 +91,4 @@
     <xacro:wheelR prefix="front"/>
     <xacro:wheelR prefix="rear"/>
-    <xacro:macro name="bin" params = "prefix">
-        <link name = "bin_${prefix}">
-            <visual>
-                <origin xyz="0 0 0" rpy = "0 0 0"/>
-                <geometry>
-                    <mesh filename = "file://$(find mobile_bot)/meshes/mobile_bot/bin.obj"/>
-                </geometry>
-                <material name = "red"/>
-            </visual>
-            <collision>
-                <origin xyz = "0 0 0" rpy = "0 0 0"/>
-                <geometry>
-                    <mesh filename = "file://$(find mobile_bot)/meshes/mobile_bot/bin.obj"/>
-                </geometry>
-                <material name = "red"/>
-            </collision>
-            <inertial>
-                <origin xyz = "0 0 0" rpy="0 0 0"/>
-                <mass value = "0.200"/>
-                <inertia
-                    ixx = "0.004" ixy="0.00" ixz="0.00"
-                    iyy = "0.004" iyz="0.0"
-                    izz = "0.004"/>
-            </inertial>
-        </link>
-    </xacro:macro>
-    <xacro:bin prefix="red"/>
-    <xacro:bin prefix="green"/>
     <xacro:macro name= "camera" params="prefix">
         <link name = "camera_${prefix}">
@@ -198,16 +170,4 @@
         <axis xyz="-1 0 0"/>
     </joint>
-    <joint name= "bin_joint_one" type="fixed">
-        <origin xyz="0.185 -0.15 0.231" rpy="${PI/2} 0 0"/>
-        <parent link = "chassis"/>
-        <child link = "bin_red"/>
-        <axis xyz = "1 0 0"/>
-    </joint>
-    <joint name= "bin_joint_two" type="fixed">
-        <origin xyz="-0.185 -0.15 0.231" rpy="${PI/2} 0 0"/>
-        <parent link = "chassis"/>
-        <child link = "bin_green"/>
-        <axis xyz = "1 0 0"/>
-    </joint>
     <joint name= "camera_joint" type="fixed">
         <origin xyz="0.0 0.395 0.074" rpy="${-PI/2} 0 0"/>

Commit message: minor changes

File: urdf/mobile.urdf (robot description, URDF)
Before this commit: robot mobile_bot, 10 links, 9 joints
Joints:
- joint base_link_joint: origin xyz=0 0 0.15 rpy=0 0 1.5707963267948966 -> xyz=0 0 0.118 rpy=0 0 0
- joint front_left_wheel_joint: origin xyz=-0.273 0.2237 -0.12 rpy=0 0 0 -> xyz=-0.273 0.2237 0 rpy=0 0 0; parent chassis -> base_footprint
- joint front_right_wheel_joint: origin xyz=0.273 0.2237 -0.12 rpy=0 0 0 -> xyz=0.273 0.2237 0 rpy=0 0 0; parent chassis -> base_footprint
- joint rear_left_wheel_joint: origin xyz=-0.273 -0.2237 -0.12 rpy=0 0 0 -> xyz=-0.273 -0.2237 0 rpy=0 0 0; parent chassis -> base_footprint
- joint rear_right_wheel_joint: origin xyz=0.273 -0.2237 -0.12 rpy=0 0 0 -> xyz=0.273 -0.2237 0 rpy=0 0 0; parent chassis -> base_footprint

File: urdf/mobile.urdf.xacro (robot description, xacro)
@@ -8,11 +8,4 @@
     <xacro:include filename ="$(find mobile_bot)/urdf/gazebo_description/physics.gazebo"/>
     <xacro:include filename ="$(find mobile_bot)/urdf/mobile.ros2_control"/>
-    <!--########################################################################################-->
-    <link name = "base_footprint"></link>
-    <joint name="base_link_joint" type="fixed">
-        <origin xyz="0 0 0.15" rpy="0 0 ${PI/2}"/>
-        <parent link= "base_footprint"/>
-        <child link = "chassis"/>
-        <axis xyz="0 0 0"/>
-    </joint>
+    <!--############################################################################################-->
 </robot>

File: urdf/mobile_bot.urdf.xacro (robot description, xacro)
@@ -10,4 +10,6 @@
     <material name="white"><color rgba="0.9 0.9 0.9 1.0"/></material>
     <material name="black"><color rgba="0.15 0.15 0.15 1.0"/></material>
+    <link name = "base_footprint">
+    </link>
     <link name = "chassis">
         <visual>
@@ -146,25 +148,31 @@
     </link>
     <!--###################### JOINTS ########################-->
+    <joint name="base_link_joint" type="fixed">
+        <origin xyz="0 0 0.118" rpy="0 0 0"/>
+        <parent link= "base_footprint"/>
+        <child link = "chassis"/>
+        <axis xyz="0 0 0"/>
+    </joint>
     <joint name="front_left_wheel_joint" type ="continuous">
-        <origin xyz="-0.273 0.2237 -0.12" rpy="0 0 0"/>
-        <parent link = "chassis"/>
+        <origin xyz="-0.273 0.2237 0" rpy="0 0 0"/>
+        <parent link = "base_footprint"/>
         <child link = "right_front_wheel"/>
         <axis xyz="-1 0 0 "/>
     </joint>
     <joint name="rear_left_wheel_joint" type ="continuous">
-        <origin xyz="-0.273 -0.2237 -0.12" rpy="0 0 0"/>
-        <parent link = "chassis"/>
+        <origin xyz="-0.273 -0.2237 0" rpy="0 0 0"/>
+        <parent link = "base_footprint"/>
         <child link = "left_rear_wheel"/>
         <axis xyz="-1 0 0"/>
     </joint>
     <joint name="front_right_wheel_joint" type ="continuous">
-        <origin xyz="0.273 0.2237 -0.12" rpy="0 0 0"/>
-        <parent link = "chassis"/>
+        <origin xyz="0.273 0.2237 0" rpy="0 0 0"/>
+        <parent link = "base_footprint"/>
         <child link = "left_front_wheel"/>
         <axis xyz="-1 0 0"/>
     </joint>
     <joint name="rear_right_wheel_joint" type ="continuous">
-        <origin xyz="0.273 -0.2237 -0.12" rpy="0 0 0"/>
-        <parent link = "chassis"/>
+        <origin xyz="0.273 -0.2237 0" rpy="0 0 0"/>
+        <parent link = "base_footprint"/>
         <child link = "right_rear_wheel"/>
         <axis xyz="-1 0 0"/>
